File: kicad/pcb_stm32.kicad_pcb (KiCad board)
At the start: 2 copper layers, 9 parts, among them J1 PRESET, J2 PROBE, J3 ESP-01S, J4 DISP_PORT, SW1 SW_SPST

Commit message: A few fixes
Parts:
- added BZ1: Buzzer, Buzzer_Beeper:Buzzer_12x9.5RM7.6, F.Cu at (94.0, 26.0)
- added C1: 100 nF, Capacitor_SMD:C_0603_1608Metric, F.Cu at (101.9, 23.6)
- added C2: 100 nF, Capacitor_SMD:C_0603_1608Metric, F.Cu at (101.9, 19.0)
- BT1, SW1: footprint TerminalBlock_Phoenix:TerminalBlock_Phoenix_MKDS-1,5-2-5.08_1x02_P5.08mm_Horizontal -> Connector_JST:JST_XH_B2B-XH-A_1x02_P2.50mm_Vertical
- J1, J2: footprint Connector_PinHeader_2.54mm:PinHeader_1x02_P2.54mm_Vertical -> Connector_JST:JST_XH_B2B-XH-A_1x02_P2.50mm_Vertical
- J4: footprint Connector_PinHeader_2.54mm:PinHeader_1x04_P2.54mm_Vertical -> Connector_JST:JST_XH_B4B-XH-A_1x04_P2.50mm_Vertical
- moved SW1 70.0 mm to (55.1, 33.0), turned to 180 degrees
- moved R2 65.3 mm to (101.3, 15.7)
- moved J2 63.3 mm to (105.9, 17.3)
- moved BT1 59.7 mm to (55.1, 40.6), turned to 180 degrees
- moved J1 52.6 mm to (105.9, 24.4)
- moved R1 52.1 mm to (101.3, 26.9)
- moved J4 43.2 mm to (83.7, 24.8), turned to 90 degrees
- moved J3 41.9 mm to (78.7, 17.1)
- moved A1 7.01 mm to (67.3, 46.4)
Connections:
- A1 pad 12: ESP_GPIO2 -> BUZZ
- A1 pad 18: +3V3 -> (no net)
- A1 pad 29: (no net) -> GND
- A1 pad 4: (no net) -> GND
- A1 pad 7: (no net) -> ESP_GPIO2
- J3 pad 1: ESP_TX -> +3V3
- J3 pad 2: GND -> ESP_RX
- J3 pad 3: ESP_CH_PD -> ESP_RST
- J3 pad 4: ESP_GPIO2 -> ESP_GIO0
- J3 pad 5: ESP_RST -> ESP_CH_PD
- J3 pad 6: ESP_GIO0 -> ESP_GPIO2
- J3 pad 7: +3V3 -> ESP_TX
- J3 pad 8: ESP_RX -> GND
- SW1 pad 1: Net-(BT1-Pad2) -> VCC
- SW1 pad 2: VCC -> Net-(BT1-Pad2)
Routing:
- net +3V3: track 0.00 -> 68.3 mm
- net ESP_GIO0: track 0.00 -> 64.0 mm
- net ESP_GPIO2: track 0.00 -> 42.4 mm
- net ESP_RX: track 0.00 -> 33.9 mm
- net ESP_RST: track 0.00 -> 28.2 mm
- net ESP_CH_PD: track 0.00 -> 25.7 mm
- net ADC2: track 0.00 -> 25.4 mm
- net ESP_TX: track 0.00 -> 25.3 mm
- net BUZZ: track 0.00 -> 23.0 mm
- net ADC1: track 0.00 -> 16.5 mm
- net DPY_SDA: track 0.00 -> 15.1 mm
- net DPY_SCK: track 0.00 -> 13.0 mm
- net VCC: track 0.00 -> 13.0 mm
- net Net-(BT1-Pad2): track 0.00 -> 7.62 mm
- net GND: track 0.00 -> 3.02 mm, vias 0 -> 1
- added copper zone on B.Cu, net GND
Other:
- board outline added: 63.1 x 35.3 mm
- board text added: "Rev 1.2"
