File: kicad/pcb_stm32.sch (KiCad schematic (older format))
At the start: 9 parts, among them J1 PRESET, J2 PROBE, J3 ESP-01S, J4 DISP_PORT, SW1 SW_SPST

Commit message: A few fixes
Parts:
- added BZ1: Buzzer, Buzzer_Beeper:Buzzer_12x9.5RM7.6, symbol Device:Buzzer
- added C1, C2: 100 nF, Capacitor_SMD:C_0603_1608Metric, symbol Device:C
- BT1, SW1: footprint TerminalBlock_Phoenix:TerminalBlock_Phoenix_MKDS-1,5-2-5.08_1x02_P5.08mm_Horizontal -> Connector_JST:JST_PH_B2B-PH-K_1x02_P2.00mm_Vertical
- J1, J2: footprint Connector_PinHeader_2.54mm:PinHeader_1x02_P2.54mm_Vertical -> Connector_JST:JST_PH_B2B-PH-K_1x02_P2.00mm_Vertical
- J3: footprint Connector_PinSocket_2.54mm:PinSocket_2x04_P2.54mm_Horizontal -> Connector_PinSocket_2.54mm:PinSocket_2x04_P2.54mm_Vertical
- J4: footprint Connector_PinHeader_2.54mm:PinHeader_1x04_P2.54mm_Vertical -> Connector_JST:JST_PH_B4B-PH-K_1x04_P2.00mm_Vertical
Connections:
- net +3V3: now also J3.1 (Pin_1); no longer A1.18 (AREF), J3.7 (Pin_7)
- net ADC1: now also C1.2
- net ADC2: now also C2.2
- net DPY_SCK: now also A1.24 (A5); no longer A1.8 (D5)
- net DPY_SDA: now also A1.23 (A4); no longer A1.7 (D4)
- net ESP_CH_PD: now also J3.5 (Pin_5); no longer J3.3 (Pin_3)
- net ESP_GIO0: now also J3.4 (Pin_4); no longer J3.6 (Pin_6)
- net ESP_GPIO2: now also A1.7 (D4), J3.6 (Pin_6); no longer A1.12 (D9), J3.4 (Pin_4)
- net ESP_RST: now also J3.3 (Pin_3); no longer J3.5 (Pin_5)
- net ESP_RX: now also J3.2 (Pin_2); no longer J3.8 (Pin_8)
- net ESP_TX: now also J3.7 (Pin_7); no longer J3.1 (Pin_1)
- net GND: now also A1.29 (GND), A1.4 (GND), J3.8 (Pin_8), BZ1.2 (+), C1.1, C2.1; no longer J3.2 (Pin_2)
- net VCC: now also SW1.1 (A); no longer SW1.2 (B)
- net at BT1.2 (-): now also SW1.2 (B); no longer SW1.1 (A)
- new net BUZZ: A1.12 (D9), BZ1.1 (-)
- no-connect marks 17 -> 15
Other:
- moved on the sheet: J1, J2, R1, R2, SW1
